File: Quansheng_UV-K5_PCB_R51-V1.4 (1).kicad_sch (KiCad schematic)
At the start: 515 parts, among them J1 USB_C_Receptacle_USB2.0, J2 Conn_Batt_K5, J4 Conn_Coaxial_K5, J5 SJ1-3525N (3.5mm), J6 Connector_Jack_2.5mm_PJ-204, Q1 2SC4226, Q10 Si2301DS, Q11 2SC3052, Q12 DTC114E, Q13 DTC114E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

Commit message: es8311 driver
Parts:
- C77: value 120u -> 120n
Changed lines of the file:
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@@
 			)
 		)
-		(property "Value" "120u"
+		(property "Value" "120n"
 			(at 143.383 310.134 90)
 			(effects
